File: LOF.kicad_pcb (KiCad board)
At the start: 4 copper layers, 63 parts, among them IC10 PEL12D-4225S-S1024, IC11 PEL12D-4225S-S1024, IC12 PEL12D-4225S-S1024, IC13 PEL12D-4225S-S1024, IC14 PEL12D-4225S-S1024, IC15 PEL12D-4225S-S1024, IC16 PEL12D-4225S-S1024, IC9 PEL12D-4225S-S1024, J1 Conn_01x01, J10 Conn_01x01, J11 Conn_01x01, J12 Conn_01x01, J13 Conn_01x01, J14 Conn_01x01, J15 Conn_01x01, J16 Conn_01x01, J17 Conn_01x01, J18 Conn_01x01, J19 Conn_01x01, J2 Conn_01x01, J20 Conn_01x01, J21 Conn_01x01, J22 Conn_01x01, J23 Conn_01x01, J24 Conn_01x01, J25 Conn_01x01, J3 Conn_01x01, J4 Conn_01x01, J5 Conn_01x01, J6 Conn_01x01, J7 Conn_01x01, J8 Conn_01x01, J9 Conn_01x01

Commit message: PCB Ready
Parts:
- removed A1: RaspberryPi_Pico, Module:RaspberryPi_Pico_Common_Unspecified
- added H1: MountingHole, MountingHole:MountingHole_3.2mm_M3_Pad, F.Cu at (55.5, 55.5)
- added H2: MountingHole, MountingHole:MountingHole_3.2mm_M3_Pad, F.Cu at (225.5, 55.5)
- added H3: MountingHole, MountingHole:MountingHole_3.2mm_M3, F.Cu at (225.5, 142.5)
- added H4: MountingHole, MountingHole:MountingHole_3.2mm_M3, F.Cu at (55.5, 142.5)
- added J26: M20-7822046, SamacSys_Parts:RHDR20W70P0X254_1X20_5120X250X865P, B.Cu at (180.5, 65.6)
- added J27: M20-7822046, SamacSys_Parts:RHDR20W70P0X254_1X20_5120X250X865P, B.Cu at (180.5, 83.4)
- C1, C10, C11, C12, C13, C14, C15, C16, C2, C3, C4, C5, C6, C7, C8, C9: footprint Kicad Libs:CAPC3216X90N -> SamacSys_Parts:CAPC3216X90N; moved to B.Cu
- IC10, IC11, IC12, IC13, IC14, IC15, IC16, IC9: footprint Kicad Libs:PEL12D4225SS1024 -> SamacSys_Parts:PEL12D4225SS1024
- J1, J10, J11, J12, J13, J14, J15, J16, J17, J18, J19, J2, J20, J21, J22, J23, J24, J25, J3, J4, J5, J6, J7, J8, J9, R1, R2, RN9: moved to B.Cu
- moved J23 317.7 mm to (225.5, 68.9)
- moved J24 316.7 mm to (225.5, 65.4)
- moved J25 315.9 mm to (225.5, 61.9)
- moved R2 288.5 mm to (205.4, 64.0), turned to -90 degrees
- moved C16 284.2 mm to (62.9, 117.2), turned to 180 degrees
- moved R1 283.2 mm to (201.1, 64.0), turned to -90 degrees
- moved C8 270.2 mm to (76.4, 117.2)
- moved C12 266.8 mm to (62.9, 89.3), turned to 180 degrees
- moved C15 261.0 mm to (90.4, 117.2), turned to 180 degrees
- moved C4 251.4 mm to (76.4, 89.3)
- moved C7 247.9 mm to (103.9, 117.2)
- moved C11 242.1 mm to (90.4, 89.3), turned to 180 degrees
- moved C14 238.6 mm to (118.0, 117.2), turned to 180 degrees
- moved C3 227.3 mm to (103.9, 89.3)
- moved RN8 225.9 mm to (176.2, 132.5), turned to -90 degrees
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Connections:
- C1 pad 1: /AOut1 -> /A_Out1
- C10 pad 1: /BOut2 -> /B_Out2
- C11 pad 1: /BOut3 -> /B_Out3
- C12 pad 1: /BOut4 -> /B_Out4
- C13 pad 1: /BOut5 -> /B_Out5
- C14 pad 1: /BOut6 -> /B_Out6
- C15 pad 1: /BOut7 -> /B_Out7
- C16 pad 1: /BOut8 -> /B_Out8
- C2 pad 1: /AOut2 -> /A_Out2
- C3 pad 1: /AOut3 -> /A_Out3
- C4 pad 1: /AOut4 -> /A_Out4
- C5 pad 1: /AOut5 -> /A_Out5
- C6 pad 1: /AOut6 -> /A_Out6
- C7 pad 1: /AOut7 -> /A_Out7
- C8 pad 1: /AOut8 -> /A_Out8
- C9 pad 1: /BOut1 -> /B_Out1
- IC10 pad 2: /PWM_9 -> /PWM_3
- IC10 pad 3: /PWM_8 -> /PWM_2
- IC10 pad A1: /AOut5 -> /RC Filtered Encoders/encoders1/AIn2
- IC10 pad B1: /BOut5 -> /RC Filtered Encoders/encoders1/BIn2
- IC11 pad 2: /PWM_3 -> /PWM_5
- IC11 pad 3: /PWM_2 -> /PWM_4
- IC11 pad A1: /AOut2 -> /RC Filtered Encoders/encoders1/AIn3
- IC11 pad B1: /BOut2 -> /RC Filtered Encoders/encoders1/BIn3
- IC12 pad 2: /PWM_10 -> /PWM_7
- IC12 pad 3: /PWM_11 -> /PWM_6
- IC12 pad A1: /AOut6 -> /RC Filtered Encoders/encoders1/AIn4
- IC12 pad B1: /BOut6 -> /RC Filtered Encoders/encoders1/BIn4
- IC13 pad 2: /PWM_5 -> /PWM_9
- IC13 pad 3: /PWM_4 -> /PWM_8
- IC13 pad A1: /AOut3 -> /RC Filtered Encoders/encoders1/AIn5
- IC13 pad B1: /BOut3 -> /RC Filtered Encoders/encoders1/BIn5
- IC14 pad 2: /PWM_12 -> /PWM_11
- IC14 pad 3: /PWM_13 -> /PWM_10
- IC14 pad A1: /AOut7 -> /RC Filtered Encoders/encoders1/AIn6
- IC14 pad B1: /BOut7 -> /RC Filtered Encoders/encoders1/BIn6
- IC15 pad 2: /PWM_7 -> /PWM_13
- IC15 pad 3: /PWM_6 -> /PWM_12
- IC15 pad A1: /AOut4 -> /RC Filtered Encoders/encoders1/AIn7
- IC15 pad B1: /BOut4 -> /RC Filtered Encoders/encoders1/BIn7
- IC16 pad A1: /AOut8 -> /RC Filtered Encoders/encoders1/AIn8
- IC16 pad B1: /BOut8 -> /RC Filtered Encoders/encoders1/BIn8
- IC9 pad A1: /AOut1 -> /RC Filtered Encoders/encoders1/AIn1
- IC9 pad B1: /BOut1 -> /RC Filtered Encoders/encoders1/BIn1
- J1 pad 1: /3V3 -> /LED_VCC
- J2 pad 1: /LED_VCC -> /3V3
- RN5 pad 10: /AOut7 -> /RC Filtered Encoders/encoders1/AIn7
- RN5 pad 11: /AOut6 -> /RC Filtered Encoders/encoders1/AIn6
- RN5 pad 12: /AOut5 -> /RC Filtered Encoders/encoders1/AIn5
- RN5 pad 13: /AOut4 -> /RC Filtered Encoders/encoders1/AIn4
- RN5 pad 14: /AOut3 -> /RC Filtered Encoders/encoders1/AIn3
- RN5 pad 15: /AOut2 -> /RC Filtered Encoders/encoders1/AIn2
- RN5 pad 16: /AOut1 -> /RC Filtered Encoders/encoders1/AIn1
- RN5 pad 9: /AOut8 -> /RC Filtered Encoders/encoders1/AIn8
- RN6 pad 10: /BOut7 -> /RC Filtered Encoders/encoders1/BIn7
- RN6 pad 11: /BOut6 -> /RC Filtered Encoders/encoders1/BIn6
- RN6 pad 12: /BOut5 -> /RC Filtered Encoders/encoders1/BIn5
- RN6 pad 13: /BOut4 -> /RC Filtered Encoders/encoders1/BIn4
- RN6 pad 14: /BOut3 -> /RC Filtered Encoders/encoders1/BIn3
- RN6 pad 15: /BOut2 -> /RC Filtered Encoders/encoders1/BIn2
- RN6 pad 16: /BOut1 -> /RC Filtered Encoders/encoders1/BIn1
- RN6 pad 9: /BOut8 -> /RC Filtered Encoders/encoders1/BIn8
- RN7 pad 1: /AOut1 -> /RC Filtered Encoders/encoders1/AIn1
- RN7 pad 10: /AOut7 -> /A_Out7
- RN7 pad 11: /AOut6 -> /A_Out6
- RN7 pad 12: /AOut5 -> /A_Out5
- RN7 pad 13: /AOut4 -> /A_Out4
- RN7 pad 14: /AOut3 -> /A_Out3
- RN7 pad 15: /AOut2 -> /A_Out2
- RN7 pad 16: /AOut1 -> /A_Out1
- RN7 pad 2: /AOut2 -> /RC Filtered Encoders/encoders1/AIn2
- RN7 pad 3: /AOut3 -> /RC Filtered Encoders/encoders1/AIn3
- RN7 pad 4: /AOut4 -> /RC Filtered Encoders/encoders1/AIn4
- RN7 pad 5: /AOut5 -> /RC Filtered Encoders/encoders1/AIn5
- RN7 pad 6: /AOut6 -> /RC Filtered Encoders/encoders1/AIn6
- RN7 pad 7: /AOut7 -> /RC Filtered Encoders/encoders1/AIn7
- RN7 pad 8: /AOut8 -> /RC Filtered Encoders/encoders1/AIn8
- RN7 pad 9: /AOut8 -> /A_Out8
- RN8 pad 1: /BOut1 -> /RC Filtered Encoders/encoders1/BIn1
- RN8 pad 10: /BOut7 -> /B_Out7
- RN8 pad 11: /BOut6 -> /B_Out6
- RN8 pad 12: /BOut5 -> /B_Out5
- RN8 pad 13: /BOut4 -> /B_Out4
- RN8 pad 14: /BOut3 -> /B_Out3
- RN8 pad 15: /BOut2 -> /B_Out2
- RN8 pad 16: /BOut1 -> /B_Out1
- RN8 pad 2: /BOut2 -> /RC Filtered Encoders/encoders1/BIn2
- RN8 pad 3: /BOut3 -> /RC Filtered Encoders/encoders1/BIn3
- RN8 pad 4: /BOut4 -> /RC Filtered Encoders/encoders1/BIn4
- RN8 pad 5: /BOut5 -> /RC Filtered Encoders/encoders1/BIn5
- RN8 pad 6: /BOut6 -> /RC Filtered Encoders/encoders1/BIn6
- RN8 pad 7: /BOut7 -> /RC Filtered Encoders/encoders1/BIn7
- RN8 pad 8: /BOut8 -> /RC Filtered Encoders/encoders1/BIn8
- RN8 pad 9: /BOut8 -> /B_Out8
- RN9 pad 15: /SCL -> /SDA
- RN9 pad 16: /SDA -> /SCL
- S1 pad 3: /GPIO18 -> /GPIO21
- S2 pad 3: /GPIO19 -> /GPIO20
- S3 pad 3: /GPIO20 -> /GPIO19
- S4 pad 3: /GPIO21 -> /GPIO18
Routing:
- net /3V3: track 0.00 -> 291.2 mm, vias 0 -> 4
- net /B_Out8: track 0.00 -> 224.9 mm, vias 0 -> 2
- net /RC Filtered Encoders/encoders1/AIn8: track 0.00 -> 196.0 mm
- net /A_Out8: track 0.00 -> 182.1 mm, vias 0 -> 2
- net /LED_VCC: track 0.00 -> 181.3 mm
- net /RC Filtered Encoders/encoders1/AIn4: track 0.00 -> 178.0 mm
- net /OE: track 0.00 -> 173.5 mm
- net /SDA: track 0.00 -> 172.0 mm
- net /SCL: track 0.00 -> 171.7 mm
- net /B_Out4: track 0.00 -> 167.7 mm, vias 0 -> 2
- net /B_Out7: track 0.00 -> 167.2 mm, vias 0 -> 3
- net /B_Out3: track 0.00 -> 156.6 mm, vias 0 -> 3
- net /RC Filtered Encoders/encoders1/AIn3: track 0.00 -> 150.0 mm
- net /A_Out3: track 0.00 -> 141.2 mm, vias 0 -> 1
- net /A_Out4: track 0.00 -> 140.2 mm, vias 0 -> 2
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- added copper zone on B.Cu, net GND
Other:
- board outline added: 180 x 97 mm
