File: LOF.kicad_sch (KiCad schematic)
At the start: 35 parts, among them J1 Conn_01x01, J10 Conn_01x01, J11 Conn_01x01, J12 Conn_01x01, J13 Conn_01x01, J14 Conn_01x01, J15 Conn_01x01, J16 Conn_01x01, J17 Conn_01x01, J18 Conn_01x01, J19 Conn_01x01, J2 Conn_01x01, J20 Conn_01x01, J21 Conn_01x01, J22 Conn_01x01, J23 Conn_01x01, J24 Conn_01x01, J25 Conn_01x01, J3 Conn_01x01, J4 Conn_01x01, J5 Conn_01x01, J6 Conn_01x01, J7 Conn_01x01, J8 Conn_01x01, J9 Conn_01x01

Commit message: PCB Ready
Parts:
- added H1, H2: MountingHole, MountingHole:MountingHole_3.2mm_M3_Pad, symbol Mechanical:MountingHole
- added H3, H4: MountingHole, MountingHole:MountingHole_3.2mm_M3, symbol Mechanical:MountingHole
- added J26, J27: M20-7822046, RHDR20W70P0X254_1X20_5120X250X865P, symbol SamacSys_Parts:M20-7822046
Connections:
- net 3V3: now also J2.1 (Pin_1), J26.5; no longer J1.1 (Pin_1)
- net GND: now also J26.13, J26.18, J26.3, J26.8, J27.13, J27.18, J27.3, J27.8
- net GPIO18: now also S4.3 (NC), J26.17; no longer S1.3 (NC)
- net GPIO19: now also S3.3 (NC), J26.16; no longer S2.3 (NC)
- net GPIO20: now also S2.3 (NC), J26.15; no longer S3.3 (NC)
- net GPIO21: now also S1.3 (NC), J26.14; no longer S4.3 (NC)
- net LED_VCC: now also J1.1 (Pin_1); no longer J2.1 (Pin_1)
- net OE: now also J26.12
- net SCL: now also RN9.16, J27.7; no longer RN9.15
- net SDA: now also RN9.15, J27.6; no longer RN9.16
- net VBUS: now also J26.1
- net WIPER_VR1: now also J26.10
- net WIPER_VR2: now also J26.9
- net AOut1 renamed A_Out1
- net A_Out1: now also J27.1
- net AOut2 renamed A_Out2
- net A_Out2: now also J27.4
- net AOut3 renamed A_Out3
- net A_Out3: now also J27.9
- net AOut4 renamed A_Out4
- net A_Out4: now also J27.11
- net AOut5 renamed A_Out5
- net A_Out5: now also J27.14
- net AOut6 renamed A_Out6
- net A_Out6: now also J27.16
- net AOut7 renamed A_Out7
- net A_Out7: now also J27.19
- net AOut8 renamed A_Out8
- net A_Out8: now also J26.20
- net BOut1 renamed B_Out1
- net B_Out1: now also J27.2
- net BOut2 renamed B_Out2
- net B_Out2: now also J27.5
- net BOut3 renamed B_Out3
- net B_Out3: now also J27.10
- net BOut4 renamed B_Out4
- net B_Out4: now also J27.12
- net BOut5 renamed B_Out5
- net B_Out5: now also J27.15
- net BOut6 renamed B_Out6
- net B_Out6: now also J27.17
- net BOut7 renamed B_Out7
- net B_Out7: now also J27.20
- net BOut8 renamed B_Out8
- net B_Out8: now also J26.19
- no-connect marks 18 -> 23
Other:
- sheet RC Filtered Encoders ports: added A_Out1, A_Out2, A_Out3, A_Out4, A_Out5, A_Out6, A_Out7, A_Out8, B_Out1, B_Out2, B_Out3, B_Out4, B_Out5, B_Out6, B_Out7, B_Out8; removed AOut1, AOut2, AOut3, AOut4, AOut5, AOut6, AOut7, AOut8, BOut1, BOut2, BOut3, BOut4, BOut5, BOut6, BOut7, BOut8
- moved on the sheet: A1, J1, J10, J11, J12, J13, J14, J15, J16, J17, J18, J19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
