File: encoder.kicad_sch (KiCad schematic)
At the start: 8 parts, among them IC10 PEL12D-4225S-S1024, IC11 PEL12D-4225S-S1024, IC12 PEL12D-4225S-S1024, IC13 PEL12D-4225S-S1024, IC14 PEL12D-4225S-S1024, IC15 PEL12D-4225S-S1024, IC16 PEL12D-4225S-S1024, IC9 PEL12D-4225S-S1024

Commit message: Added rest of the encoder terminal to hierarchical sheets
Connections:
- net GND: no longer IC10.4 (COM), IC11.4 (COM), IC12.4 (COM), IC13.4 (COM), IC14.4 (COM), IC15.4 (COM), IC16.4 (COM), IC9.4 (COM)
- new net E1_SW: IC9.4 (COM)
- new net E2_SW: IC11.4 (COM)
- new net E3_SW: IC13.4 (COM)
- new net E4_SW: IC15.4 (COM)
- new net E5_SW: IC10.4 (COM)
- new net E6_SW: IC12.4 (COM)
- new net E7_SW: IC14.4 (COM)
- new net E8_SW: IC16.4 (COM)

Commit message: Made fixes according to the erc
Connections:
- net E1_SW is gone; now on net GND: IC9.4 (COM)
- net E2_SW is gone; now on net GND: IC11.4 (COM)
- net E3_SW is gone; now on net GND: IC13.4 (COM)
- net E4_SW is gone; now on net GND: IC15.4 (COM)
- net E5_SW is gone; now on net GND: IC10.4 (COM)
- net E6_SW is gone; now on net GND: IC12.4 (COM)
- net E7_SW is gone; now on net GND: IC14.4 (COM)
- net E8_SW is gone; now on net GND: IC16.4 (COM)

Commit message: PCB Ready
Parts:
- renumbered IC11 to IC10, IC13 to IC11, IC15 to IC12, IC10 to IC13, IC12 to IC14, IC14 to IC15
